Commit message: Add a camera transform and enable landmarks.

File: cartographer_mir/urdf/mir-100.urdf (robot description, URDF)
Before this commit: robot mir-100, 6 links, 5 joints
Links:
- added link camera; visual box size=0.06 0.04 0.02
Joints:
- added joint camera_joint: type fixed, parent base_link, child camera, origin xyz=0.439636 0 0.57 rpy=0 1.57 0
